Commit message: added mug to simulation

File: robotarm_simulation/urdf/mug.urdf (robot description, URDF)
Before this commit: robot myfirst, 1 links, 0 joints
Links:
- link base_link: geometry visual cylinder length=0.04 radius=0.02

Commit message: added cup location & grabbing checks

File: robotarm_simulation/urdf/mug.urdf (robot description, URDF)
Before this commit: robot mug, 1 links, 0 joints
Links:
- removed link base_link
- added link mug_link; visual cylinder length=0.04 radius=0.02
